Commit message: Added Kinect2 to Robot Description

File: sawyer_description/urdf/sawyer.urdf.xacro (robot description, xacro)
@@ -6,4 +6,5 @@
   <xacro:arg name="electric_gripper" default="false"/>
   <!-- Sawyer Base URDF -->
+    <xacro:include filename="$(find kinect2_description)/urdf/kinect2.urdf.xacro"/>
   <xacro:include filename="$(find sawyer_description)/urdf/sawyer_base.urdf.xacro">
     <xacro:arg name="gazebo" value="${gazebo}"/>

File: sawyer_description/urdf/sawyer_base.urdf.xacro (robot description, xacro)
@@ -532,3 +532,6 @@
     <axis xyz="0 0 0"/>
   </joint>
+  <xacro:kinect2_xacro prefix="head" parent="head">
+    <origin xyz=".04 -.095 .3" rpy="${radians(-90-30)} 0 ${radians(-90)}"/>
+</xacro:kinect2_xacro>
 </robot>
