Commit message: Updated sawyer.xacro, rviz config and launch file

File: sawyer_description/urdf/sawyer_base.urdf.xacro (robot description, xacro)
@@ -533,5 +533,5 @@
   </joint>
   <xacro:kinect2_xacro prefix="head" parent="head">
-    <origin xyz=".04 -.095 .3" rpy="${radians(-90-30)} 0 ${radians(-90)}"/>
+    <origin xyz=".04 -.09 .3" rpy="${radians(-90-30)} 0 ${radians(-90)}"/>
 </xacro:kinect2_xacro>
 </robot>
